File: projects/ESC/ESC.brd (EAGLE design)
At the start: 139.7 x 38.1 mm, 91 parts, among them J1 1755529, J2 1755529, J3 1755529, J4 1755529, U1 STM32F405RGT6, U10 CSD88584Q5DCT, U11 CSD88584Q5DCT, U12 CSD88584Q5DCT, U13 CSD88584Q5DCT, U2 CSD88584Q5DCT, U3 CSD88584Q5DCT, U4 CSD88584Q5DCT, U5 CSD88584Q5DCT, U6 CSD88584Q5DCT, U7 CSD88584Q5DCT, U8 CSD88584Q5DCT, U9 CSD88584Q5DCT, Y1 ECS-80-S-4X

Commit message: some later things to do
Parts:
- removed U$7: SAMTEC, VESC_SHIT:SAMTEC
- added C6: 0.1uF, SparkFun-Capacitors:0603
- added R6: 1.5k, SparkFun-Resistors:0603
- added U14: SN74CBTLV3257PWR, SN74CBTLV3257PWR:SN74CBTLV3257PWR
- U$5: value SAMTEC -> ESC2BACKPLANE; device VESC_SHIT:SAMTEC -> ESC_to_Backplane_Connectors:ESC2BACKPLANE_WHOLE
- moved R1 131.6 mm to (58.9, 8.89), flipped to the bottom, turned to 90 degrees
- moved R2 130.2 mm to (57.1, 8.89), flipped to the bottom, turned to 90 degrees
- moved C41 125.0 mm to (58.2, 22.9)
- moved C16 121.4 mm to (60.2, 14.2), flipped to the bottom, turned to 270 degrees
- moved GREEN_LED 114.8 mm to (58.9, 5.59), flipped to the bottom, turned to 90 degrees
- moved RED_LED 111.0 mm to (57.1, 5.59), flipped to the bottom, turned to 90 degrees
- moved R4 101.6 mm to (99.8, 11.2), flipped to the bottom, turned to 90 degrees
- moved C30 100.8 mm to (68.3, 3.81), flipped to the bottom, turned to 90 degrees
- moved C18 99.4 mm to (110.5, 6.10), turned to 180 degrees
- moved C20 99.4 mm to (115.6, 3.56)
- moved C21 98.5 mm to (113.0, 4.32), turned to 270 degrees
- moved C19 93.3 mm to (108.7, 11.9), flipped to the bottom
- moved R17 92.4 mm to (106.9, 15.5), flipped to the bottom, turned to 180 degrees
- moved R15 92.2 mm to (116.1, 15.5), flipped to the bottom
- moved R16 91.6 mm to (110.0, 15.5), flipped to the bottom, turned to 180 degrees
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Connections:
- removed net 12V: U$5.P1-1, U$5.P1-2, U$5.P1-3, U$5.P1-4, U$5.P1-5, U$5.P1-6, U$5.P1-7, U$5.P1-8, U$5.P2-1, U$5.P2-2, U$5.P2-3, U$5.P2-4, U$5.P2-5, U$5.P2-6, U$5.P2-7, U$5.P2-8, U$5.P3-1, U$5.P3-2, U$5.P3-3, U$5.P3-4, U$5.P3-5, U$5.P3-6, U$5.P3-7, U$5.P3-8, U$5.P4-1, U$5.P4-2, U$5.P4-3, U$5.P4-4, U$5.P4-5, U$5.P4-6, U$5.P4-7, U$5.P4-8
- removed net 3V3: U$5.1, U$5.10, U$5.11, U$5.12, U$5.13, U$5.14, U$5.15, U$5.16, U$5.17, U$5.18, U$5.19, U$5.2, U$5.20, U$5.21, U$5.22, U$5.23, U$5.24, U$5.3, U$5.4, U$5.5, U$5.6, U$5.7, U$5.8, U$5.9, U1.1, U1.13, U1.19, U1.32, U1.48, U1.64
- removed net N$11: U$2.27
- removed net N$14: U$2.29
- removed net N$20: U$3.25
- removed net N$21: U$3.27
- removed net N$22: U$3.29
- removed net N$37: U$4.25
- removed net N$38: U$4.27
- removed net N$39: U$4.29
- removed net SLC_1B: U4.12, U4.13, U4.14, U4.15, U4.16, U4.17, U4.18, U4.19, U4.20
- new net +12V: U$5.P$10, U$5.P$11, U$5.P$12, U$5.P$13, U$5.P$23, U$5.P$24, U$5.P$25, U$5.P$26, U$5.P$27, U$5.P$9, U$5.P$A, U$5.P$B, U$5.P$C, U$5.P$D, U$5.P$E, U$5.P$O, U$5.P$P, U$5.P$Q, U$5.P$R, U$5.P$S
- new net NRST_IN: U14.P$9
- new net PROG_SEL: U$5.P$5
- new net S: U$6.S, U14.P$1
- new net SWCLK_IN: U14.P$4
- new net SWDIO_IN: U14.P$7
- net +3V3: now also C6.1, R6.2, U$5.P$G, U$5.P$H, U$5.P$U, U$5.P$V, U1.1, U1.13, U1.19, U1.32, U1.48, U1.64, U14.P$16
- net CAN_H: now also U$5.P$6; no longer U$7.24
- net CAN_L: now also U$5.P$7; no longer U$7.23
- net EN_3: now also U1.55; no longer U1.54
- net FAULT_1: now also U$2.17
- net FAULT_2: now also U$1.17
- net FAULT_3: now also U$3.17, U1.54; no longer U1.55
- net FAULT_4: now also U$4.17
- net GND: now also C6.2, U$5.P$1, U$5.P$15, U$5.P$16, U$5.P$17, U$5.P$18, U$5.P$2, U$5.P$3, U$5.P$4, U$5.P$AA, U$5.P$BB, U$5.P$J, U$5.P$K, U$5.P$L, U$5.P$M, U$5.P$N, U$5.P$X, U$5.P$Y, U$5.P$Z, U14.P$8; no longer U$7.P1-1, U$7.P1-2, U$7.P1-3, U$7.P1-4, U$7.P1-5, U$7.P1-6, U$7.P1-7, U$7.P1-8, U$7.P2-1, U$7.P2-2, U$7.P2-3, U$7.P2-4, U$7.P2-5, U$7.P2-6, U$7.P2-7, U$7.P2-8, U$7.P3-1, U$7.P3-2, U$7.P3-3, U$7.P3-4, U$7.P3-5, U$7.P3-6, U$7.P3-7, U$7.P3-8, U$7.P4-1, U$7.P4-2, U$7.P4-3, U$7.P4-4, U$7.P4-5, U$7.P4-6, U$7.P4-7, U$7.P4-8
- net INHA_1: now also U$2.25
- net INHA_3: now also U$3.25, U1.56; no longer U1.53
- net INHA_4: now also U$4.25, U1.50; no longer U1.59
- net INHB_1: now also U$2.27
- net INHB_3: now also U$3.27, U1.57; no longer U1.52
- net INHB_4: now also U$4.27, U1.51; no longer U1.58
- net INHC_1: now also U$2.29
- net INHC_2: now also U$1.29
- net INHC_3: now also U$3.29, U1.59; no longer U$1.29, U1.51
- net INHC_4: now also U$4.29, U1.53; no longer U1.57
- net INL_3: now also U1.58; no longer U1.50
- net INL_4: now also U1.52; no longer U1.56
- net N$10: now also R6.1, U14.P$15; no longer U$2.25
- net NRST: now also U14.P$11
- net SLB_1: now also U4.12, U4.13, U4.14, U4.15, U4.16, U4.17, U4.18, U4.19, U4.20
- net SWCLK: now also U14.P$2
- net SWDIO: now also U14.P$5
Routing:
- net VM_2: track 70.8 -> 0.00 mm, vias 6 -> 0
- net VM_3: track 0.00 -> 66.3 mm
- net +3V3: track 0.00 -> 45.8 mm, vias 0 -> 5
- net SLA_2: track 36.0 -> 0.00 mm
- net SHA_2: track 30.5 -> 0.00 mm, vias 2 -> 0
- net GLA_2: track 28.6 -> 0.00 mm
- net GHA_2: track 26.2 -> 0.00 mm
- net CAN_H: track 35.0 -> 9.49 mm
- net PHASE_C4: track 4.00 -> 29.1 mm
- net DVDD_2: track 24.9 -> 0.00 mm, vias 2 -> 0
- net EN_2: track 24.8 -> 0.00 mm, vias 1 -> 0
- net SLB_2: track 24.4 -> 0.00 mm, vias 2 -> 0
- net SLC_2: track 18.9 -> 0.00 mm
- net GLB_2: track 18.5 -> 0.00 mm, vias 2 -> 0
- net SHB_2: track 18.3 -> 0.00 mm
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- removed copper zone on layer 1, net 12V
- removed copper zone on layer 1, net 12V1
- removed copper zone on layer 1, net 3V3
