File: Test/test.sch (EAGLE design)
At the start: 47 parts, among them J2 1755529, U1 STM32F405RGT6, U2 CSD88584Q5DCT, U3 CSD88584Q5DCT, U4 CSD88584Q5DCT, Y1 ECS-80-S-4X

Commit message: couple improvements to the board and datasheets
Parts:
- added J1: 284512-3, ThrusterConnector:284512-3
- added U$1: MURATA-DC-DC, MURATA_3pin_dcdc:MURATA-DC-DC
- C11: value 4.7uF -> 20[F
- C2: value 4.7uF -> 20pF
- R3, R5: value 1k -> 0
- RESET1: value SWITCH -> (none); device DiscreteComponents:SWITCH -> Push button - FSM2JMTR:DISCRETECOMPONENTS_SWITCH
Connections:
- net 12V: now also U$1.VIN
- net 3V3: now also SV1.8, U$1.VOUT; no longer SV1.6
- net CAN_H: now also SV1.3; no longer SV1.5
- net CAN_L: now also SV1.2; no longer SV1.4
- net GND: now also SV1.6, U$1.GND; no longer SV1.7
- net NRST: now also SV1.4; no longer SV1.8
- net PHASE_A1: now also J1.3
- net PHASE_B1: now also J1.2
- net PHASE_C1: now also J1.1
- net SWCLK: now also SV1.7; no longer SV1.3
- net SWDIO: now also SV1.5; no longer SV1.2

Commit message: grounded drain of low side fets and other improvements
Parts:
- removed U$6: TCAN337D, PI_Shield_Library:TCAN337D
- added U$3: TCAN337D, STM and CAN parts:TCAN337D
- C10: value 4.7uF -> 0.1uF
- C30: value 4.7uF -> 0.1IuF
- R1, R2: value 1k -> 470
- R4: value 1k -> 10k
Connections:
- net N$1 renamed LED1
- net N$2 renamed LED1_MID
- net N$3 renamed LED2_MID
- net N$4 renamed LED2
- removed net INL_1: U$2G$1.INLA, U$2G$1.INLB, U$2G$1.INLC, U1.PB12
- removed net SLA_1: U$2G$1.SLA, U3.PGND, U3.PGND_2, U3.PGND_3, U3.PGND_4, U3.PGND_5, U3.PGND_6, U3.PGND_7, U3.PGND_8, U3.PGND_9
- removed net SLB_1: U$2G$1.SLB, U4.PGND, U4.PGND_2, U4.PGND_3, U4.PGND_4, U4.PGND_5, U4.PGND_6, U4.PGND_7, U4.PGND_8, U4.PGND_9
- removed net SLC_1: U$2G$1.SLC, U2.PGND, U2.PGND_2, U2.PGND_3, U2.PGND_4, U2.PGND_5, U2.PGND_6, U2.PGND_7, U2.PGND_8, U2.PGND_9
- new net INLA_1: U$2G$1.INLA, U1.PB12
- new net INLB_1: U$2G$1.INLB
- new net INLC_1: U$2G$1.INLC
- net 3V3: now also U$3.VCC; no longer U$6.VCC
- net CAN_H: now also U$3.CANH; no longer U$6.CANH
- net CAN_L: now also U$3.CANL; no longer U$6.CANL
- net CAN_RX: now also U$3.RXD; no longer U$6.RXD
- net CAN_TX: now also U$3.TXD; no longer U$6.TXD
- net GND: now also U$2G$1.SLA, U$2G$1.SLB, U$2G$1.SLC, U$3.GND, U2.PGND, U2.PGND_2, U2.PGND_3, U2.PGND_4, U2.PGND_5, U2.PGND_6, U2.PGND_7, U2.PGND_8, U2.PGND_9, U3.PGND, U3.PGND_2, U3.PGND_3, U3.PGND_4, U3.PGND_5, U3.PGND_6, U3.PGND_7, U3.PGND_8, U3.PGND_9, U4.PGND, U4.PGND_2, U4.PGND_3, U4.PGND_4, U4.PGND_5, U4.PGND_6, U4.PGND_7, U4.PGND_8, U4.PGND_9; no longer U$6.GND
Other:
- note added: "SLA_1"
- note added: "SLB_1"
- note added: "SLC_1"
- note added: "TODO: Break out the INL(B/C)_1 pins for PWM"
- moved on the sheet: C15, C30, GREEN_LED, R1, R2, R8, R9, RED_LED

Commit message: progress
Parts:
- removed GREEN_LED, RED_LED: TLMS1100-GS08, VESC_SHIT:TLMS1100-GS08
- removed J2: 1755529, VESC_SHIT:1755529
- removed U2, U3, U4: CSD88584Q5DCT, VESC_SHIT:CSD88584Q5DCT
- added D1: RED, LED-0805:LED-0805
- added D2: GREEN, LED-0805:LED-0805
- added JP2, JP4, JP6: JUMPER-SMT_2_NC_TRACE_SILK, SparkFun-Jumpers:JUMPER-SMT_2_NC_TRACE_SILK
- added Q1, Q2, Q3: (no value), Dual NMOS:DUAL-NMOS
- added U$4: 3PINCONNECTOR, afro_20A_esc:3PINCONNECTOR
- C11: value 20[F -> 20pF
- U$2: device VESC_SHIT:DRV8320H -> Motor Driver - DRV8320HRTVT:DRV8320H
- U1: value STM32F405RGT6 -> (none); device VESC_SHIT:STM32F405RGT6 -> STM32F405RGT6:STM32F405RGT6
Connections:
- net DVDD_1 renamed 3V3_OUT
- net N$16 renamed CPL
- net N$17 renamed IDRIVE
- net N$18 renamed MODE
- net N$34 renamed V_CAP_L
- net N$9 renamed CPH
- removed net SHA_1: U$2G$1.SHA, U3.SH
- removed net SHB_1: U$2G$1.SHB, U4.SH
- removed net SHC_1: U$2G$1.SHC, U2.SH
- new net DLA_1: JP2.1
- new net DLB_1: JP4.1
- new net DLC_1: JP6.1
- net 12V: now also Q1G$2.D1, Q1G$2.D2, Q2G$1.D1, Q2G$1.D2, Q3G$1.D1, Q3G$1.D2; no longer U2.VIN, U3.VIN, U4.VIN
- net GHA_1: now also Q1G$2.G; no longer U3.GH
- net GHB_1: now also Q2G$1.G; no longer U4.GH
- net GHC_1: now also Q3G$1.G; no longer U2.GH
- net GLA_1: now also Q1G$1.G; no longer U3.GL
- net GLB_1: now also Q2G$2.G; no longer U4.GL
- net GLC_1: now also Q3G$2.G; no longer U2.GL
- net GND: now also D1.C, D2.C, Q1G$1.S, Q2G$2.S, Q3G$2.S; no longer GREEN_LED.1, RED_LED.1, U2.PGND, U2.PGND_2, U2.PGND_3, U2.PGND_4, U2.PGND_5, U2.PGND_6, U2.PGND_7, U2.PGND_8, U2.PGND_9, U3.PGND, U3.PGND_2, U3.PGND_3, U3.PGND_4, U3.PGND_5, U3.PGND_6, U3.PGND_7, U3.PGND_8, U3.PGND_9, U4.PGND, U4.PGND_2, U4.PGND_3, U4.PGND_4, U4.PGND_5, U4.PGND_6, U4.PGND_7, U4.PGND_8, U4.PGND_9
- net LED1_MID: now also D1.A; no longer GREEN_LED.2
- net LED2_MID: now also D2.A; no longer RED_LED.2
- net PHASE_A1: now also JP2.2, Q1G$1.D1, Q1G$1.D2, Q1G$2.S, U$2G$1.SHA, U$4.A; no longer J2.1, U3.VSW, U3.VSW_2, U3.VSW_3, U3.VSW_4, U3.VSW_5, U3.VSW_6, U3.VSW_7, U3.VSW_8, U3.VSW_9
- net PHASE_B1: now also JP4.2, Q2G$1.S, Q2G$2.D1, Q2G$2.D2, U$2G$1.SHB, U$4.B; no longer J2.2, U4.VSW, U4.VSW_2, U4.VSW_3, U4.VSW_4, U4.VSW_5, U4.VSW_6, U4.VSW_7, U4.VSW_8, U4.VSW_9
- net PHASE_C1: now also JP6.2, Q3G$1.S, Q3G$2.D1, Q3G$2.D2, U$2G$1.SHC, U$4.C; no longer J2.3, U2.VSW, U2.VSW_2, U2.VSW_3, U2.VSW_4, U2.VSW_5, U2.VSW_6, U2.VSW_7, U2.VSW_8, U2.VSW_9
Other:
- note added: "Consider switching to the DRV8340"
- note added: "SHA_1"
- note added: "SHB_1"
- note added: "SHC_1"
