File: projects/Test/test.brd (EAGLE design)
At the start: 65.8 x 27.6 mm, 48 parts, among them J1 284512-3, Y1 ECS-80-S-4X

Commit message: fixed errors
Parts:
- moved R4 0.96 mm to (55.1, 12.9)
- moved R11 0.85 mm to (28.3, 3.49)
- moved C13 0.78 mm to (31.5, 22.7)
- moved R10 0.55 mm to (26.4, 3.37)
- moved C10 0.26 mm to (56.2, 10.4)
- moved RESET1 0.06 mm to (56.1, 10.9)
Routing:
- net NRST: track 21.9 -> 28.8 mm, vias 2 -> 3
- net +3V3: track 49.5 -> 48.0 mm
- net SOA: track 24.5 -> 23.2 mm, vias 3 -> 2
- net CPL: track 3.14 -> 4.27 mm
- net PHASE_A1: track 31.2 -> 32.3 mm
- net INLB_1: track 20.9 -> 21.7 mm
- net CPH: track 2.62 -> 3.33 mm
- net VDS: track 9.28 -> 9.93 mm
