File: projects/Test/test.sch (EAGLE design)
At the start: 93 parts, among them J1 1755529, J2 1755529, J3 1755529, J4 1755529, U1 STM32F405RGT6, U10 CSD88584Q5DCT, U11 CSD88584Q5DCT, U12 CSD88584Q5DCT, U13 CSD88584Q5DCT, U14 SN74CBTLV3257PWR, U2 CSD88584Q5DCT, U3 CSD88584Q5DCT, U4 CSD88584Q5DCT, U5 CSD88584Q5DCT, U6 CSD88584Q5DCT, U7 CSD88584Q5DCT, U8 CSD88584Q5DCT, U9 CSD88584Q5DCT, Y1 ECS-80-S-4X

Commit message: some later things to do
Parts:
- removed C18, C22, C26: 47nF, SparkFun-Capacitors:47NF-0603-25V-5%
- removed C19, C21, C23, C25, C27, C29: 1.0uF, SparkFun-Capacitors:1.0UF-0603-16V-10%
- removed C20, C24, C28, C6: 0.1uF, SparkFun-Capacitors:0.1UF-0603-25V-(+80/-20%)
- removed J1, J3, J4: 1755529, VESC_SHIT:1755529
- removed R13, R18, R23: 47k, rcl:R-US_R0603
- removed R14, R15, R16, R17, R19, R20, R21, R22, R24, R25, R26, R27: (no value), rcl:R-US_R0603
- removed R6: 1.5k, SparkFun-Resistors:1.5KOHM-0603-1/10W-1%
- removed SV2: (no value), con-lsta:FE05-1
- removed U$1, U$3, U$4: DRV8320H, VESC_SHIT:DRV8320H
- removed U$5: ESC2BACKPLANE, ESC_to_Backplane_Connectors:ESC2BACKPLANE
- removed U10, U11, U12, U13, U5, U6, U7, U8, U9: CSD88584Q5DCT, VESC_SHIT:CSD88584Q5DCT
- removed U14: SN74CBTLV3257PWR, SN74CBTLV3257PWR:SN74CBTLV3257PWR
- added SV1: (no value), con-lsta:FE08-1
Connections:
- removed net +12V: U$5G$1.P$10, U$5G$1.P$11, U$5G$1.P$12, U$5G$1.P$13, U$5G$1.P$23, U$5G$1.P$24, U$5G$1.P$25, U$5G$1.P$26, U$5G$1.P$27, U$5G$1.P$9, U$5G$2.P$A, U$5G$2.P$B, U$5G$2.P$C, U$5G$2.P$D, U$5G$2.P$E, U$5G$2.P$O, U$5G$2.P$P, U$5G$2.P$Q, U$5G$2.P$R, U$5G$2.P$S
- removed net +3V3: C12.1, C16.1, C30.1, C32.1, C33.1, C34.1, C35.1, C38.1, C39.1, C4.1, C40.1, C41.1, C5.1, C6.1, R4.2, R6.2, SV2.5, U$5G$2.P$G, U$5G$2.P$H, U$5G$2.P$U, U$5G$2.P$V, U$6.VCC, U1.VBAT, U1.VDDA, U1.VDD_1, U1.VDD_2, U1.VDD_3, U1.VDD_4, U14.VCC
- removed net DVDD_2: C23.1, R19.2, R21.2, U$1G$2.DVDD
- removed net DVDD_3: C19.1, R14.2, R16.2, U$3G$2.DVDD
- removed net DVDD_4: C27.1, R24.2, R26.2, U$4G$2.DVDD
- removed net EN_2: U$1G$1.ENABLE, U1.PA10
- removed net EN_3: U$3G$1.ENABLE, U1.PB3
- removed net EN_4: U$4G$1.ENABLE, U1.PB1
- removed net FAULT_2: U$1G$1.FAULT_N, U1.PA11
- removed net FAULT_3: U$3G$1.FAULT_N, U1.PD2
- removed net FAULT_4: U$4G$1.FAULT_N, U1.PB2
- removed net GHA_2: U$1G$1.GHA, U6.GH
- removed net GHA_3: U$3G$1.GHA, U9.GH
- removed net GHA_4: U$4G$1.GHA, U12.GH
- removed net GHB_2: U$1G$1.GHB, U5.GH
- removed net GHB_3: U$3G$1.GHB, U8.GH
- removed net GHB_4: U$4G$1.GHB, U11.GH
- removed net GHC_2: U$1G$1.GHC, U7.GH
- removed net GHC_3: U$3G$1.GHC, U10.GH
- removed net GHC_4: U$4G$1.GHC, U13.GH
- removed net GLA_2: U$1G$1.GLA, U6.GL
- removed net GLA_3: U$3G$1.GLA, U9.GL
- removed net GLA_4: U$4G$1.GLA, U12.GL
- removed net GLB_2: U$1G$1.GLB, U5.GL
- removed net GLB_3: U$3G$1.GLB, U8.GL
- removed net GLB_4: U$4G$1.GLB, U11.GL
- removed net GLC_2: U$1G$1.GLC, U7.GL
- removed net GLC_3: U$3G$1.GLC, U10.GL
- removed net GLC_4: U$4G$1.GLC, U13.GL
- removed net IDRIVE: R19.1, R20.2, U$1G$1.IDRIVE
- removed net INHA_2: U$1G$1.INHA, U1.PA9
- removed net INHA_3: U$3G$1.INHA, U1.PB4
- removed net INHA_4: U$4G$1.INHA, U1.PA15
- removed net INHB_2: U$1G$1.INHB, U1.PA8
- removed net INHB_3: U$3G$1.INHB, U1.PB5
- removed net INHB_4: U$4G$1.INHB, U1.PC10
- removed net INHC_2: U$1G$1.INHC, U1.PC9
- removed net INHC_3: U$3G$1.INHC, U1.PB7
- removed net INHC_4: U$4G$1.INHC, U1.PC12
- removed net INL_3: U$3G$1.INLA, U$3G$1.INLB, U$3G$1.INLC, U1.PB6
- removed net INL_4: U$4G$1.INLA, U$4G$1.INLB, U$4G$1.INLC, U1.PC11
- removed net N$10: R6.1, U14.OE
- removed net N$23: C21.1, U$3G$2.VCP
- removed net N$24: C18.1, U$3G$1.CPH
- removed net N$25: C18.2, U$3G$1.CPL
- removed net N$26: R14.1, R15.2, U$3G$1.IDRIVE
- removed net N$27: R13.2, U$3G$1.MODE
- removed net N$28: R16.1, R17.2, U$3G$1.VDS
- removed net N$30: C25.1, U$1G$2.VCP
- removed net N$31: C22.1, U$1G$1.CPH
- removed net N$32: C22.2, U$1G$1.CPL
- removed net N$35: R18.2, U$1G$1.MODE
- removed net N$40: C29.1, U$4G$2.VCP
- removed net N$41: C26.1, U$4G$1.CPH
- removed net N$42: C26.2, U$4G$1.CPL
- removed net N$43: R24.1, R25.2, U$4G$1.IDRIVE
- removed net N$44: R23.2, U$4G$1.MODE
- removed net N$45: R26.1, R27.2, U$4G$1.VDS
- removed net NRST_IN: U14.3A
- removed net PHASE_A2: J1.1, U6.VSW, U6.VSW_2, U6.VSW_3, U6.VSW_4, U6.VSW_5, U6.VSW_6, U6.VSW_7, U6.VSW_8, U6.VSW_9
- removed net PHASE_A3: J3.1, U9.VSW, U9.VSW_2, U9.VSW_3, U9.VSW_4, U9.VSW_5, U9.VSW_6, U9.VSW_7, U9.VSW_8, U9.VSW_9
- removed net PHASE_A4: J4.1, U12.VSW, U12.VSW_2, U12.VSW_3, U12.VSW_4, U12.VSW_5, U12.VSW_6, U12.VSW_7, U12.VSW_8, U12.VSW_9
- removed net PHASE_B2: J1.2, U5.VSW, U5.VSW_2, U5.VSW_3, U5.VSW_4, U5.VSW_5, U5.VSW_6, U5.VSW_7, U5.VSW_8, U5.VSW_9
- removed net PHASE_B3: J3.2, U8.VSW, U8.VSW_2, U8.VSW_3, U8.VSW_4, U8.VSW_5, U8.VSW_6, U8.VSW_7, U8.VSW_8, U8.VSW_9
- removed net PHASE_B4: J4.2, U11.VSW, U11.VSW_2, U11.VSW_3, U11.VSW_4, U11.VSW_5, U11.VSW_6, U11.VSW_7, U11.VSW_8, U11.VSW_9
- removed net PHASE_C2: J1.3, U7.VSW, U7.VSW_2, U7.VSW_3, U7.VSW_4, U7.VSW_5, U7.VSW_6, U7.VSW_7, U7.VSW_8, U7.VSW_9
- removed net PHASE_C3: J3.3, U10.VSW, U10.VSW_2, U10.VSW_3, U10.VSW_4, U10.VSW_5, U10.VSW_6, U10.VSW_7, U10.VSW_8, U10.VSW_9
- removed net PHASE_C4: J4.3, U13.VSW, U13.VSW_2, U13.VSW_3, U13.VSW_4, U13.VSW_5, U13.VSW_6, U13.VSW_7, U13.VSW_8, U13.VSW_9
- removed net PROG_SEL: U$5G$1.P$5
- removed net S: U$6.S, U14.S
- removed net SHA_2: U$1G$1.SHA, U6.SH
- removed net SHA_3: U$3G$1.SHA, U9.SH
- removed net SHA_4: U$4G$1.SHA, U12.SH
- removed net SHB_2: U$1G$1.SHB, U5.SH
- removed net SHB_3: U$3G$1.SHB, U8.SH
- removed net SHB_4: U$4G$1.SHB, U11.SH
- removed net SHC_2: U$1G$1.SHC, U7.SH
- removed net SHC_3: U$3G$1.SHC, U10.SH
- removed net SHC_4: U$4G$1.SHC, U13.SH
- removed net SLA_2: U$1G$1.SLA, U6.PGND, U6.PGND_2, U6.PGND_3, U6.PGND_4, U6.PGND_5, U6.PGND_6, U6.PGND_7, U6.PGND_8, U6.PGND_9
- removed net SLA_3: U$3G$1.SLA, U9.PGND, U9.PGND_2, U9.PGND_3, U9.PGND_4, U9.PGND_5, U9.PGND_6, U9.PGND_7, U9.PGND_8, U9.PGND_9
- removed net SLA_4: U$4G$1.SLA, U12.PGND, U12.PGND_2, U12.PGND_3, U12.PGND_4, U12.PGND_5, U12.PGND_6, U12.PGND_7, U12.PGND_8, U12.PGND_9
- removed net SLB_2: U$1G$1.SLB, U5.PGND, U5.PGND_2, U5.PGND_3, U5.PGND_4, U5.PGND_5, U5.PGND_6, U5.PGND_7, U5.PGND_8, U5.PGND_9
- removed net SLB_3: U$3G$1.SLB, U8.PGND, U8.PGND_2, U8.PGND_3, U8.PGND_4, U8.PGND_5, U8.PGND_6, U8.PGND_7, U8.PGND_8, U8.PGND_9
- removed net SLB_4: U$4G$1.SLB, U11.PGND, U11.PGND_2, U11.PGND_3, U11.PGND_4, U11.PGND_5, U11.PGND_6, U11.PGND_7, U11.PGND_8, U11.PGND_9
- removed net SLC_2: U$1G$1.SLC, U7.PGND, U7.PGND_2, U7.PGND_3, U7.PGND_4, U7.PGND_5, U7.PGND_6, U7.PGND_7, U7.PGND_8, U7.PGND_9
- removed net SLC_3: U$3G$1.SLC, U10.PGND, U10.PGND_2, U10.PGND_3, U10.PGND_4, U10.PGND_5, U10.PGND_6, U10.PGND_7, U10.PGND_8, U10.PGND_9
- removed net SLC_4: U$4G$1.SLC, U13.PGND, U13.PGND_2, U13.PGND_3, U13.PGND_4, U13.PGND_5, U13.PGND_6, U13.PGND_7, U13.PGND_8, U13.PGND_9
- removed net SWCLK_IN: U14.1A
- removed net SWDIO_IN: U14.2A
- removed net VDS: R21.1, R22.2, U$1G$1.VDS
- removed net VM_1: C15.1, C17.2, U$2G$1.VDRAIN, U$2G$2.VM, U2.VIN, U3.VIN, U4.VIN
- removed net VM_2: C24.1, C25.2, U$1G$1.VDRAIN, U$1G$2.VM, U5.VIN, U6.VIN, U7.VIN
- removed net VM_3: C20.1, C21.2, U$3G$1.VDRAIN, U$3G$2.VM, U10.VIN, U8.VIN, U9.VIN
- removed net VM_4: C28.1, C29.2, U$4G$1.VDRAIN, U$4G$2.VM, U11.VIN, U12.VIN, U13.VIN
- new net 12V: C15.1, C17.2, SV1.1, U$2G$1.VDRAIN, U$2G$2.VM, U2.VIN, U3.VIN, U4.VIN
- new net 3V3: C12.1, C16.1, C30.1, C32.1, C33.1, C34.1, C35.1, C38.1, C39.1, C4.1, C40.1, C41.1, C5.1, R4.2, SV1.6, U$6.VCC, U1.VBAT, U1.VDDA, U1.VDD_1, U1.VDD_2, U1.VDD_3, U1.VDD_4
- net CAN_H: now also SV1.5; no longer U$5G$1.P$6
- net CAN_L: now also SV1.4; no longer U$5G$1.P$7
- net GND: now also SV1.7; no longer C19.2, C20.2, C23.2, C24.2, C27.2, C28.2, C6.2, R13.1, R15.1, R17.1, R18.1, R20.1, R22.1, R23.1, R25.1, R27.1, SV2.3, U$1G$2.AGND, U$1G$2.PAD, U$1G$2.PGND, U$3G$2.AGND, U$3G$2.PAD, U$3G$2.PGND, U$4G$2.AGND, U$4G$2.PAD, U$4G$2.PGND, U$5G$1.P$1, U$5G$1.P$15, U$5G$1.P$16, U$5G$1.P$17, U$5G$1.P$18, U$5G$1.P$2, U$5G$1.P$3, U$5G$1.P$4, U$5G$2.P$AA, U$5G$2.P$BB, U$5G$2.P$J, U$5G$2.P$K, U$5G$2.P$L, U$5G$2.P$M, U$5G$2.P$N, U$5G$2.P$X, U$5G$2.P$Y, U$5G$2.P$Z, U14.GND
- net INL_2: no longer U$1G$1.INLA, U$1G$1.INLB, U$1G$1.INLC
- net NRST: now also SV1.8; no longer SV2.1, U14.3B1
- net SWCLK: now also SV1.3; no longer SV2.4, U14.1B1
- net SWDIO: now also SV1.2; no longer SV2.2, U14.2B1

Commit message: some changes i made a while back and forgot to push
Parts:
- added R12, R13, R6: (no value), resistor-shunt:PMD
Connections:
- net GND: now also R12.2, R13.2, R6.2
- net SLA_1: now also R6.1
- net SLB_1: now also R12.1
- net SLC_1: now also R13.1
Changed lines of the file:
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@@
 <part name="U4" library="VESC_SHIT" library_urn="urn:adsk.eagle:library:11793053" deviceset="CSD88584Q5DCT" device=""/>
 <part name="U3" library="VESC_SHIT" library_urn="urn:adsk.eagle:library:11793053" deviceset="CSD88584Q5DCT" device=""/>
+<part name="R6" library="resistor-shunt" library_urn="urn:adsk.eagle:library:346" deviceset="PMD" device="" package3d_urn="urn:adsk.eagle:package:25216/1"/>
+<part name="R12" library="resistor-shunt" library_urn="urn:adsk.eagle:library:346" deviceset="PMD" device="" package3d_urn="urn:adsk.eagle:package:25216/1"/>
+<part name="R13" library="resistor-shunt" library_urn="urn:adsk.eagle:library:346" deviceset="PMD" device="" package3d_urn="urn:adsk.eagle:package:25216/1"/>
+<part name="GND12" library="SparkFun-PowerSymbols" library_urn="urn:adsk.eagle:library:530" deviceset="GND" device=""/>
+<part name="GND13" library="SparkFun-PowerSymbols" library_urn="urn:adsk.eagle:library:530" deviceset="GND" device=""/>
+<part name="GND14" library="SparkFun-PowerSymbols" library_urn="urn:adsk.eagle:library:530" deviceset="GND" device=""/>
 </parts>
 <sheets>
@@
 <attribute name="VALUE" x="50.5206" y="110.7186" size="2.0828" layer="96" ratio="6" rot="SR0"/>
 </instance>
+<instance part="R6" gate="G$1" x="55.88" y="43.18" smashed="yes" rot="R90">
+<attribute name="NAME" x="54.5084" y="39.37" size="1.778" layer="95" rot="R90"/>
+<attribute name="VALUE" x="58.801" y="39.37" size="1.778" layer="96" rot="R90"/>
+</instance>
+<instance part="R12" gate="G$1" x="127" y="43.18" smashed="yes" rot="R90">
+<attribute name="NAME" x="125.6284" y="39.37" size="1.778" layer="95" rot="R90"/>
+<attribute name="VALUE" x="129.921" y="39.37" size="1.778" layer="96" rot="R90"/>
+</instance>
+<instance part="R13" gate="G$1" x="200.66" y="40.64" smashed="yes" rot="R90">
+<attribute name="NAME" x="199.2884" y="36.83" size="1.778" layer="95" rot="R90"/>
+<attribute name="VALUE" x="203.581" y="36.83" size="1.778" layer="96" rot="R90"/>
+</instance>
+<instance part="GND12" gate="1" x="55.88" y="35.56" smashed="yes">
+<attribute name="VALUE" x="55.88" y="35.306" size="1.778" layer="96" align="top-center"/>
+</instance>
+<instance part="GND13" gate="1" x="127" y="35.56" smashed="yes">
+<attribute name="VALUE" x="127" y="35.306" size="1.778" layer="96" align="top-center"/>
+</instance>
+<instance part="GND14" gate="1" x="200.66" y="33.02" smashed="yes">
+<attribute name="VALUE" x="200.66" y="32.766" size="1.778" layer="96" align="top-center"/>
+</instance>
 </instances>
 <busses>
@@
 <junction x="73.66" y="83.82"/>
 <pinref part="U3" gate="A" pin="PGND"/>
+<pinref part="R6" gate="G$1" pin="1"/>
 </segment>
 </net>
@@
 <junction x="144.78" y="83.82"/>
 <pinref part="U4" gate="A" pin="PGND"/>
+<pinref part="R12" gate="G$1" pin="1"/>
 </segment>
 </net>
@@
 <junction x="218.44" y="83.82"/>
 <pinref part="U2" gate="A" pin="PGND"/>
+<pinref part="R13" gate="G$1" pin="1"/>
 </segment>
 </net>
@@
 </segment>
 </net>
+<net name="GND" class="0">
+<segment>
+<pinref part="GND12" gate="1" pin="GND"/>
+<pinref part="R6" gate="G$1" pin="2"/>
+</segment>
+<segment>
+<pinref part="GND13" gate="1" pin="GND"/>
+<pinref part="R12" gate="G$1" pin="2"/>
+</segment>
+<segment>
+<pinref part="GND14" gate="1" pin="GND"/>
+<pinref part="R13" gate="G$1" pin="2"/>
+</segment>
+</net>

Commit message: Consolidate test boards to one place
Parts:
- removed GREEN_LED, RED_LED: TLMS1100-GS08, VESC_SHIT:TLMS1100-GS08
- removed J2: 1755529, VESC_SHIT:1755529
- removed R12, R13, R6: (no value), resistor-shunt:PMD
- removed U$6: TCAN337D, PI_Shield_Library:TCAN337D
- removed U2, U3, U4: CSD88584Q5DCT, VESC_SHIT:CSD88584Q5DCT
- added D1: RED, LED-0805:LED-0805
- added D2: GREEN, LED-0805:LED-0805
- added J1: 284512-3, ThrusterConnector:284512-3
- added JP2, JP4, JP6: JUMPER-SMT_2_NC_TRACE_SILK, SparkFun-Jumpers:JUMPER-SMT_2_NC_TRACE_SILK
- added Q1, Q2, Q3: (no value), Dual NMOS:DUAL-NMOS
- added U$1: MURATA-DC-DC, MURATA_3pin_dcdc:MURATA-DC-DC
- added U$3: TCAN337D, STM and CAN parts:TCAN337D
- added U$4: 3PINCONNECTOR, afro_20A_esc:3PINCONNECTOR
- C10: value 4.7uF -> 0.1uF
- C11, C2: value 4.7uF -> 20pF
- C30: value 4.7uF -> 0.1IuF
- R1, R2: value 1k -> 470
- R3, R5: value 1k -> 0
- R4: value 1k -> 10k
- RESET1: value SWITCH -> (none); device DiscreteComponents:SWITCH -> Push button - FSM2JMTR:DISCRETECOMPONENTS_SWITCH
- U$2: device VESC_SHIT:DRV8320H -> Motor Driver - DRV8320HRTVT:DRV8320H
- U1: value STM32F405RGT6 -> (none); device VESC_SHIT:STM32F405RGT6 -> STM32F405RGT6:STM32F405RGT6
Connections:
- net DVDD_1 renamed 3V3_OUT
- net N$1 renamed LED1
- net N$16 renamed CPL
- net N$17 renamed IDRIVE
- net N$18 renamed MODE
- net N$34 renamed V_CAP_L
- net N$4 renamed LED2
- net N$9 renamed CPH
- removed net INL_1: U$2G$1.INLA, U$2G$1.INLB, U$2G$1.INLC, U1.PB12
- removed net N$2: GREEN_LED.2, R1.1
- removed net N$3: R2.1, RED_LED.2
- removed net SHA_1: U$2G$1.SHA, U3.SH
- removed net SHB_1: U$2G$1.SHB, U4.SH
- removed net SHC_1: U$2G$1.SHC, U2.SH
- removed net SLA_1: R6.1, U$2G$1.SLA, U3.PGND, U3.PGND_2, U3.PGND_3, U3.PGND_4, U3.PGND_5, U3.PGND_6, U3.PGND_7, U3.PGND_8, U3.PGND_9
- removed net SLB_1: R12.1, U$2G$1.SLB, U4.PGND, U4.PGND_2, U4.PGND_3, U4.PGND_4, U4.PGND_5, U4.PGND_6, U4.PGND_7, U4.PGND_8, U4.PGND_9
- removed net SLC_1: R13.1, U$2G$1.SLC, U2.PGND, U2.PGND_2, U2.PGND_3, U2.PGND_4, U2.PGND_5, U2.PGND_6, U2.PGND_7, U2.PGND_8, U2.PGND_9
- new net DLA_1: JP2.1
- new net DLB_1: JP4.1
- new net DLC_1: JP6.1
- new net INLA_1: U$2G$1.INLA, U1.PB12
- new net INLB_1: U$2G$1.INLB
- new net INLC_1: U$2G$1.INLC
- new net LED1_MID: D1.A, R1.1
- new net LED2_MID: D2.A, R2.1
- net 12V: now also Q1G$2.D1, Q1G$2.D2, Q2G$1.D1, Q2G$1.D2, Q3G$1.D1, Q3G$1.D2, U$1.VIN; no longer U2.VIN, U3.VIN, U4.VIN
- net 3V3: now also SV1.8, U$1.VOUT, U$3.VCC; no longer SV1.6, U$6.VCC
- net CAN_H: now also SV1.3, U$3.CANH; no longer SV1.5, U$6.CANH
- net CAN_L: now also SV1.2, U$3.CANL; no longer SV1.4, U$6.CANL
- net CAN_RX: now also U$3.RXD; no longer U$6.RXD
- net CAN_TX: now also U$3.TXD; no longer U$6.TXD
- net GHA_1: now also Q1G$2.G; no longer U3.GH
- net GHB_1: now also Q2G$1.G; no longer U4.GH
- net GHC_1: now also Q3G$1.G; no longer U2.GH
- net GLA_1: now also Q1G$1.G; no longer U3.GL
- net GLB_1: now also Q2G$2.G; no longer U4.GL
- net GLC_1: now also Q3G$2.G; no longer U2.GL
- net GND: now also D1.C, D2.C, Q1G$1.S, Q2G$2.S, Q3G$2.S, SV1.6, U$1.GND, U$2G$1.SLA, U$2G$1.SLB, U$2G$1.SLC, U$3.GND; no longer GREEN_LED.1, R12.2, R13.2, R6.2, RED_LED.1, SV1.7, U$6.GND
- net NRST: now also SV1.4; no longer SV1.8
- net PHASE_A1: now also J1.3, JP2.2, Q1G$1.D1, Q1G$1.D2, Q1G$2.S, U$2G$1.SHA, U$4.A; no longer J2.1, U3.VSW, U3.VSW_2, U3.VSW_3, U3.VSW_4, U3.VSW_5, U3.VSW_6, U3.VSW_7, U3.VSW_8, U3.VSW_9
- net PHASE_B1: now also J1.2, JP4.2, Q2G$1.S, Q2G$2.D1, Q2G$2.D2, U$2G$1.SHB, U$4.B; no longer J2.2, U4.VSW, U4.VSW_2, U4.VSW_3, U4.VSW_4, U4.VSW_5, U4.VSW_6, U4.VSW_7, U4.VSW_8, U4.VSW_9
- net PHASE_C1: now also J1.1, JP6.2, Q3G$1.S, Q3G$2.D1, Q3G$2.D2, U$2G$1.SHC, U$4.C; no longer J2.3, U2.VSW, U2.VSW_2, U2.VSW_3, U2.VSW_4, U2.VSW_5, U2.VSW_6, U2.VSW_7, U2.VSW_8, U2.VSW_9
- net SWCLK: now also SV1.7; no longer SV1.3
- net SWDIO: now also SV1.5; no longer SV1.2
Other:
- note added: "Consider switching to the DRV8340"
- note added: "SHA_1"
- note added: "SHB_1"
- note added: "SHC_1"
- note added: "SLA_1"
- note added: "SLB_1"
- note added: "SLC_1"
- note added: "TODO: Break out the INL(B/C)_1 pins for PWM"

Commit message: Replace micro and driver. Remove CAN.
Parts:
- removed C1, C3: 2.2uF, SparkFun-Capacitors:2.2UF-0603-10V-20%
- removed C30: 0.1IuF, SparkFun-Capacitors:4.7UF0603
- removed C31: 0.1uF, SparkFun-Capacitors:0.1UF-0603-25V-(+80/-20%)
- removed C32, C33, C34, C35, C4, C40, C41, C5: 4.7uF, SparkFun-Capacitors:4.7UF0603
- removed JP2, JP4, JP6: JUMPER-SMT_2_NC_TRACE_SILK, SparkFun-Jumpers:JUMPER-SMT_2_NC_TRACE_SILK
- removed R28, R29: 60, SparkFun-Resistors:1KOHM-0603-1/10W-1%
- removed U$2: DRV8320H, Motor Driver - DRV8320HRTVT:DRV8320H
- removed U$3: TCAN337D, STM and CAN parts:TCAN337D
- removed U1: (no value), STM32F405RGT6:STM32F405RGT6
- added J10, J11: (no value), SparkFun-Connectors:BANANA_CONN
- added J2, J3, J4, J5, J6, J7, J8, J9: (no value), SparkFun-Connectors:CONN_01
- added U$5: STM32F042K6T6, STM and CAN parts:STM32F042K6T6
- added U$6: DRV8340H, Motor Driver - DRV8340H:DRV8340H
- C16, C38, C39: value 4.7uF -> 0.1uF
- R1, R2: value 470 -> 1k
- R10, R11, R8, R9: value (none) -> (none); device rcl:R-US_R0603 -> SparkFun-Resistors:RESISTOR0603
- R4: value 10k -> 1k
- R7: device rcl:R-US_R0603 -> SparkFun-Resistors:47KOHM-0603-1/10W-1%
- SV1: device con-lsta:FE08-1 -> SparkFun-Connectors:CONN_08"
Connections:
- net N$7 renamed OSC_XTAL_2
- net N$8 renamed OSC_XTAL_1
- removed net CAN_H: R28.2, SV1.3, U$3.CANH
- removed net CAN_L: R29.1, SV1.2, U$3.CANL
- removed net CAN_RX: U$3.RXD, U1.PB8
- removed net CAN_TX: U$3.TXD, U1.PB9
- removed net DLA_1: JP2.1
- removed net DLB_1: JP4.1
- removed net DLC_1: JP6.1
- removed net INL_2: U1.PC8
- removed net N$19: R10.1, R11.2, U$2G$1.VDS
- removed net N$46: C31.2, R28.1, R29.2
- removed net N$5: C1.1, U1.VSS_2
- removed net N$6: C3.1, U1.VSS_1
- new net +3V3: C12.1, C16.1, C38.1, C39.1, R4.2, U$5.VDD, U$5.VDDA, U$5.VDDIO2
- new net N$1: U$5.PB3, U$5.PB4, U$5.PB5, U$5.PB6
- new net VDS: R10.1, R11.2, U$6G$2.VDS
- net 12V: now also J10.1, J8.1, Q1G$1.D1, Q1G$1.D2, Q3G$2.D1, Q3G$2.D2, SV1.2, U$6G$1.VDRAIN, U$6G$1.VM; no longer Q1G$2.D1, Q1G$2.D2, Q3G$1.D1, Q3G$1.D2, U$2G$1.VDRAIN, U$2G$2.VM
- net 3V3: no longer C12.1, C16.1, C30.1, C32.1, C33.1, C34.1, C35.1, C38.1, C39.1, C4.1, C40.1, C41.1, C5.1, R4.2, U$3.VCC, U1.VBAT, U1.VDDA, U1.VDD_1, U1.VDD_2, U1.VDD_3, U1.VDD_4
- net 3V3_OUT: now also U$6G$1.DVDD; no longer U$2G$2.DVDD
- net CPH: now also U$6G$1.CPH; no longer U$2G$1.CPH
- net CPL: now also U$6G$1.CPL; no longer U$2G$1.CPL
- net EN_1: now also U$5.PA11, U$6G$2.ENABLE; no longer U$2G$1.ENABLE, U1.PC6
- net FAULT_1: now also U$5.PA12, U$6G$2.!FAULT; no longer U$2G$1.FAULT_N, U1.PC7
- net GHA_1: now also Q1G$1.G, U$6G$2.GHA; no longer Q1G$2.G, U$2G$1.GHA
- net GHB_1: now also U$6G$2.GHB; no longer U$2G$1.GHB
- net GHC_1: now also Q3G$2.G, U$6G$2.GHC; no longer Q3G$1.G, U$2G$1.GHC
- net GLA_1: now also Q1G$2.G, U$6G$2.GLA; no longer Q1G$1.G, U$2G$1.GLA
- net GLB_1: now also U$6G$2.GLB; no longer U$2G$1.GLB
- net GLC_1: now also Q3G$1.G, U$6G$2.GLC; no longer Q3G$2.G, U$2G$1.GLC
- net GND: now also J11.1, J9.1, Q1G$2.S, Q3G$1.S, SV1.3, U$5.PB8-BOOT0, U$5.VSS, U$6G$1.AGND, U$6G$1.PAD, U$6G$1.PGND, U$6G$2.SLA, U$6G$2.SLB, U$6G$2.SLC, U$6G$3.NC1, U$6G$3.NC10, U$6G$3.NC11, U$6G$3.NC12, U$6G$3.NC2, U$6G$3.NC3, U$6G$3.NC4, U$6G$3.NC5, U$6G$3.NC6, U$6G$3.NC7, U$6G$3.NC8, U$6G$3.NC9; no longer C1.2, C3.2, C30.2, C31.1, C32.2, C33.2, C34.2, C35.2, C4.2, C40.2, C41.2, C5.2, Q1G$1.S, Q3G$2.S, U$2G$1.SLA, U$2G$1.SLB, U$2G$1.SLC, U$2G$2.AGND, U$2G$2.PAD, U$2G$2.PGND, U$3.GND, U1.BOOT0, U1.VSSA, U1.VSS_, U1.VSS_4
- net IDRIVE: now also U$6G$2.IDRIVE; no longer U$2G$1.IDRIVE
- net INHA_1: now also J2.1, U$5.PA6, U$6G$2.INHA; no longer U$2G$1.INHA, U1.PB15
- net INHB_1: now also J3.1, U$5.PA9, U$6G$2.INHB; no longer U$2G$1.INHB, U1.PB14
- net INHC_1: now also J4.1, U$5.PA7, U$6G$2.INHC; no longer U$2G$1.INHC, U1.PB13
- net INLA_1: now also J5.1, U$5.PA8, U$6G$2.INLA; no longer U$2G$1.INLA, U1.PB12
- net INLB_1: now also J6.1, U$5.PA10, U$6G$2.INLB; no longer U$2G$1.INLB
- net INLC_1: now also J7.1, U$5.PA4, U$6G$2.INLC; no longer U$2G$1.INLC
- net LED1: now also U$5.PA0; no longer U1.PC4
- net LED2: now also U$5.PA1; no longer U1.PC5
- net MODE: now also U$6G$2.MODE; no longer U$2G$1.MODE
- net NRST: now also U$5.NRST; no longer U1.NRST
- net OSC_IN: now also U$5.PF1-OSC_OUT; no longer U1.PD0_OSC_IN
- net OSC_OUT: now also U$5.PF0-OSC_IN; no longer U1.PD1_OSC_OUT
- net PHASE_A1: now also Q1G$1.S, Q1G$2.D1, Q1G$2.D2, U$6G$2.DLA, U$6G$2.SHA; no longer JP2.2, Q1G$1.D1, Q1G$1.D2, Q1G$2.S, U$2G$1.SHA
- net PHASE_B1: now also U$6G$2.DLB, U$6G$2.SHB; no longer JP4.2, U$2G$1.SHB
- net PHASE_C1: now also Q3G$1.D1, Q3G$1.D2, Q3G$2.S, U$6G$2.DLC, U$6G$2.SHC; no longer JP6.2, Q3G$1.S, Q3G$2.D1, Q3G$2.D2, U$2G$1.SHC
- net SWCLK: now also U$5.PA14; no longer U1.PA14
- net SWDIO: now also U$5.PA13; no longer U1.PA13
- net V_CAP_L: now also U$6G$1.VCP; no longer U$2G$2.VCP
Other:
- note added: "In 1x PWM: INHA is the "carrier" wave (TIM3_CH1) INLA, INHB, and INLB control states (TIM1_CH1,2,3) INHC controls direction with hall effect sensors (unused) INLC brakes the motor (active low) (also TIM14_CH1)"
- note removed: "CAN TERMINATION"
- note removed: "CAN TRANSCEIVER"
- note removed: "Consider switching to the DRV8340"
- note removed: "Pin 19 (VDD_4)"
- note removed: "Pin 32 (VDD_1)"
- note removed: "Pin 48 (VDD_2)"
- note removed: "Pin 64 (VDD_3)"
- note removed: "TODO: Break out the INL(B/C)_1 pins for PWM"
- moved on the sheet: C10, C11, C13, C17, C2, Q1G$1, Q1G$2, Q3G$1, Q3G$2, R3, R4, R5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
